File: Ijr-X1-Core.kicad_sch (KiCad schematic)
At the start: 16 parts, among them J1 USB-C_PWR_IN, J2 USB-C_CPU_PROG, J3 USB-C_UART_BRIDGE, U1 RP2040, U2 W25Q16JVSSIQ

Commit message: Some updates
Parts:
- added C5: 100nF, symbol Device:C
- added J_GPIO: GPIO_Header_2x25, symbol Connector_Generic:Conn_02x25_Odd_Even
- added J_SWD: SWD_Debug, symbol Connector_Generic:Conn_02x03_Odd_Even
Connections:
- net GPIO27 is gone; now on net GPIO26: U1.39 (GPIO27/ADC1)
- net +3V3: now also U2.8 (VCC), J_GPIO.49 (Pin_49), J_SWD.1 (Pin_1)
- net GND: now also J3.A1 (GND), J3.A12 (GND), J3.B1 (GND), J3.B12 (GND), J3.SH (SHIELD), U2.4 (GND), J_GPIO.50 (Pin_50), J_SWD.3 (Pin_3)
- net GPIO0: now also J_GPIO.1 (Pin_1)
- net GPIO1: now also J_GPIO.2 (Pin_2)
- net GPIO10: now also J_GPIO.11 (Pin_11)
- net GPIO11: now also J_GPIO.12 (Pin_12)
- net GPIO12: now also J_GPIO.13 (Pin_13)
- net GPIO13: now also J_GPIO.14 (Pin_14)
- net GPIO14: now also J_GPIO.15 (Pin_15)
- net GPIO15: now also J_GPIO.16 (Pin_16)
- net GPIO16: now also J_GPIO.17 (Pin_17)
- net GPIO17: now also J_GPIO.18 (Pin_18)
- net GPIO18: now also J_GPIO.19 (Pin_19)
- net GPIO19: now also J_GPIO.20 (Pin_20)
- net GPIO2: now also J_GPIO.3 (Pin_3)
- net GPIO20: now also J_GPIO.21 (Pin_21)
- net GPIO21: now also J_GPIO.22 (Pin_22)
- net GPIO22: now also J_GPIO.23 (Pin_23)
- net GPIO23: now also J_GPIO.24 (Pin_24)
- net GPIO24: now also J_GPIO.25 (Pin_25)
- net GPIO25: now also J_GPIO.26 (Pin_26)
- net GPIO26: now also J_GPIO.27 (Pin_27), J_GPIO.28 (Pin_28)
- net GPIO28: now also J_GPIO.29 (Pin_29)
- net GPIO29: now also J_GPIO.30 (Pin_30)
- net GPIO3: now also J_GPIO.4 (Pin_4)
- net GPIO4: now also J_GPIO.5 (Pin_5)
- net GPIO5: now also J_GPIO.6 (Pin_6)
- net GPIO6: now also J_GPIO.7 (Pin_7)
- net GPIO7: now also J_GPIO.8 (Pin_8)
- net GPIO8: now also J_GPIO.9 (Pin_9)
- net GPIO9: now also J_GPIO.10 (Pin_10)
- net GPIO_USB_DM: now also J3.A6 (D+), J3.B6 (D+)
- net GPIO_USB_DP: now also J3.A7 (D-), J3.B7 (D-)
- net QSPI_SD2: now also U2.3 (~{WP}/IO_{2})
- net QSPI_SD3: now also U2.7 (~{HOLD}/~{RESET}/IO_{3})
- net SWD_CLK: now also J_SWD.4 (Pin_4)
- net SWD_DIO: now also J_SWD.2 (Pin_2)
- net +5V: now reaches J3.A4 (VBUS), J3.A9 (VBUS), J3.B4 (VBUS), J3.B9 (VBUS)
- net +5V: now also J1.A9 (VBUS), J1.B9 (VBUS)
- net J3_CC1: now reaches J3.A5 (CC1)
- net J3_CC2: now reaches J3.B5 (CC2)
- net J1_CC1: now reaches J1.A5 (CC1)
- no-connect marks 2 -> 24

Commit message: Some updates1
Connections:
- net +3V3: now also C5.1
- net +5V: now also C1.1, C2.1, C3.1, J2.A4 (VBUS), J2.A9 (VBUS), J2.B4 (VBUS), J2.B9 (VBUS)
- net GND: now also C1.2, C2.2, C3.2, C5.2, J1.A12 (GND), J1.B12 (GND), J1.SH (SHIELD), J2.A1 (GND), J2.A12 (GND), J2.B1 (GND), J2.B12 (GND), J2.SH (SHIELD), R1.2, R2.2, R3.2, R4.2, R5.2, R6.2; no longer R7.2
- net GPIO26: no longer J_GPIO.28 (Pin_28), U1.39 (GPIO27/ADC1)
- net J1_CC1: now also R1.1
- net J3_CC1: now also R5.1
- net J3_CC2: now also R6.1
- net RUN: now also R7.2
- net J2_CC2: now reaches R4.1
- net J2_CC2: now also J2.B5 (CC2)
- net J2_CC1: now reaches J2.A5 (CC1)
- net J2_CC1: now also R3.1
- net J2_DM: now reaches J2.A6 (D+)
- net J2_DM: now also J2.B6 (D+)
- net J2_DP: now reaches J2.A7 (D-)
- net J2_DP: now also J2.B7 (D-)
- net J1_CC2: now reaches J1.B5 (CC2)
- net J1_CC2: now also R2.1
- new net GPIO27: J_GPIO.28 (Pin_28), U1.39 (GPIO27/ADC1)
- no-connect marks 24 -> 26
Changed lines of the file:
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@@
-		(effects (font (size 1.524 1.524)))
-	)
-	(label "GND"
-		(at 111.76 71.12 0)
-		(effects (font (size 1.524 1.524)))
-	)
-	(label "RUN"
-		(at 111.76 67.31 0)
 		(effects (font (size 1.524 1.524)))
 	)
@@
 		)
 	)
-	(label "+3V3"
-		(at 113.03 95.25 0)
-		(effects (font (size 1.524 1.524)))
-	)
-	(label "GND"
-		(at 113.03 100.33 0)
-		(effects (font (size 1.524 1.524)))
-	)
 	(symbol
 		(lib_id "Connector_Generic:Conn_02x25_Odd_Even")
@@
 	)
 	(label "GPIO26"
-		(at 214.63 92.71 0)
-		(effects (font (size 1.524 1.524)))
-	)
-	(label "GPIO27"
 		(at 214.63 92.71 0)
 		(effects (font (size 1.524 1.524)))
@@
 		(effects (font (size 1.524 1.524)))
 	)
+	(label "J1_CC2"
+		(at 54.61 46.99 0)
+		(effects (font (size 1.524 1.524)))
+	)
+	(label "GND"
+		(at 39.37 57.15 0)
+		(effects (font (size 1.524 1.524)))
+	)
+	(label "GND"
+		(at 31.75 57.15 0)
+		(effects (font (size 1.524 1.524)))
+	)
+	(label "+5V"
+		(at 54.61 74.93 0)
+		(effects (font (size 1.524 1.524)))
+	)
+	(label "J2_CC1"
+		(at 54.61 80.01 0)
+		(effects (font (size 1.524 1.524)))
+	)
+	(label "J2_CC2"
+		(at 54.61 82.55 0)
+		(effects (font (size 1.524 1.524)))
+	)
+	(label "J2_DP"
+		(at 54.61 87.63 0)
+		(effects (font (size 1.524 1.524)))
+	)
+	(label "J2_DP"
+		(at 54.61 90.17 0)
+		(effects (font (size 1.524 1.524)))
+	)
+	(label "J2_DM"
+		(at 54.61 92.71 0)
+		(effects (font (size 1.524 1.524)))
+	)
+	(label "J2_DM"
+		(at 54.61 95.25 0)
+		(effects (font (size 1.524 1.524)))
+	)
+	(no_connect (at 54.61 102.87))
+	(no_connect (at 54.61 105.41))
+	(label "GND"
+		(at 39.37 113.03 0)
+		(effects (font (size 1.524 1.524)))
+	)
+	(label "GND"
+		(at 31.75 113.03 0)
+		(effects (font (size 1.524 1.524)))
+	)
+	(label "J1_CC1"
+		(at 74.93 29.21 0)
+		(effects (font (size 1.524 1.524)))
+	)
+	(label "GND"
+		(at 74.93 36.83 0)
+		(effects (font (size 1.524 1.524)))
+	)
+	(label "J1_CC2"
+		(at 74.93 40.64 0)
+		(effects (font (size 1.524 1.524)))
+	)
+	(label "GND"
+		(at 74.93 48.26 0)
+		(effects (font (size 1.524 1.524)))
+	)
+	(label "J2_CC1"
+		(at 74.93 78.74 0)
+		(effects (font (size 1.524 1.524)))
+	)
+	(label "GND"
+		(at 74.93 86.36 0)
+		(effects (font (size 1.524 1.524)))
+	)
+	(label "J2_CC2"
+		(at 74.93 91.44 0)
+		(effects (font (size 1.524 1.524)))
+	)
+	(label "GND"
+		(at 74.93 99.06 0)
+		(effects (font (size 1.524 1.524)))
+	)
+	(label "J3_CC1"
+		(at 74.93 129.54 0)
+		(effects (font (size 1.524 1.524)))
+	)
+	(label "GND"
+		(at 74.93 137.16 0)
+		(effects (font (size 1.524 1.524)))
+	)
+	(label "J3_CC2"
+		(at 74.93 140.97 0)
+		(effects (font (size 1.524 1.524)))
+	)
+	(label "GND"
+		(at 74.93 148.59 0)
+		(effects (font (size 1.524 1.524)))
+	)
+	(label "+5V"
+		(at 87.63 34.29 0)
+		(effects (font (size 1.524 1.524)))
+	)
+	(label "GND"
+		(at 87.63 41.91 0)
+		(effects (font (size 1.524 1.524)))
+	)
+	(label "+5V"
+		(at 87.63 83.82 0)
+		(effects (font (size 1.524 1.524)))
+	)
+	(label "GND"
+		(at 87.63 91.44 0)
+		(effects (font (size 1.524 1.524)))
+	)
+	(label "+5V"
+		(at 87.63 134.62 0)
+		(effects (font (size 1.524 1.524)))
+	)
+	(label "GND"
+		(at 87.63 142.24 0)
+		(effects (font (size 1.524 1.524)))
+	)
+	(label "+3V3"
+		(at 113.03 93.98 0)
+		(effects (font (size 1.524 1.524)))
+	)
+	(label "GND"
+		(at 113.03 101.6 0)
+		(effects (font (size 1.524 1.524)))
+	)
+	(label "RUN"
+		(at 111.76 71.12 0)
+		(effects (font (size 1.524 1.524)))
+	)
+	(symbol
+		(lib_id "power:PWR_FLAG")
+		(at 59.69 170.18 0)
+		(unit 1)
+		(exclude_from_sim no)
+		(in_bom yes)
+		(on_board yes)
+		(dnp no)
+		(property "Reference" "#PWR01"
+			(at 59.69 163.83 0)
+			(effects (font (size 1.27 1.27)) (hide yes))
+		)
+		(property "Value" "PWR_FLAG"
+			(at 59.69 165.1 0)
+			(effects (font (size 1.27 1.27)))
+		)
+		(property "Footprint" ""
+			(at 59.69 170.18 0)
+			(effects (font (size 1.27 1.27)) (hide yes))
+		)
+		(property "Datasheet" "~"
+			(at 59.69 170.18 0)
+			(effects (font (size 1.27 1.27)) (hide yes))
+		)
+		(instances
+			(project "Ijr-X1-Core"
+				(path "/0a8e2d86-540d-4bc7-908e-89ff2a8b35b6"
+					(reference "#PWR01") (unit 1)
+				)
+			)
+		)
+	)
 	(sheet_instances

Commit message: Some updates1
Changed lines of the file:
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@@
 		)
+	)
+	(label "+3V3"
+		(at 59.69 170.18 0)
+		(effects (font (size 1.524 1.524)))
+	)
+	(symbol
+		(lib_id "power:PWR_FLAG")
+		(at 74.93 170.18 0)
+		(unit 1)
+		(exclude_from_sim no)
+		(in_bom yes)
+		(on_board yes)
+		(dnp no)
+		(property "Reference" "#PWR02"
+			(at 74.93 163.83 0)
+			(effects (font (size 1.27 1.27)) (hide yes))
+		)
+		(property "Value" "PWR_FLAG"
+			(at 74.93 165.1 0)
+			(effects (font (size 1.27 1.27)))
+		)
+		(property "Footprint" ""
+			(at 74.93 170.18 0)
+			(effects (font (size 1.27 1.27)) (hide yes))
+		)
+		(property "Datasheet" "~"
+			(at 74.93 170.18 0)
+			(effects (font (size 1.27 1.27)) (hide yes))
+		)
+		(instances
+			(project "Ijr-X1-Core"
+				(path "/0a8e2d86-540d-4bc7-908e-89ff2a8b35b6"
+					(reference "#PWR02") (unit 1)
+				)
+			)
+		)
+	)
+	(label "GND"
+		(at 74.93 170.18 0)
+		(effects (font (size 1.524 1.524)))
 	)
 	(sheet_instances

Commit message: Some updates1
Parts:
- added J_ATX24: ATX_24Pin_Main, symbol Connector_Generic:Conn_02x12_Odd_Even
- added J_EPS8: EPS_8Pin_CPU, symbol Connector_Generic:Conn_02x04_Odd_Even
- added J_PCIE1: PCIe_6plus2_GPU1, symbol Connector_Generic:Conn_02x04_Odd_Even
- added J_PCIE2: PCIe_6plus2_GPU2, symbol Connector_Generic:Conn_02x04_Odd_Even
- added J_PWRBTN: PWR_Button, symbol Connector_Generic:Conn_01x02
- added J_PWRLED: PWR_LED, symbol Connector_Generic:Conn_01x02
- added J_PWROK: PWR_OK_TestPoint, symbol Connector_Generic:Conn_01x02
- added R8: 470R, symbol Device:R
Connections:
- net +3V3: now also J_ATX24.1 (Pin_1), J_ATX24.11 (Pin_11), J_ATX24.13 (Pin_13), J_ATX24.2 (Pin_2)
- net +5V: now also J_ATX24.21 (Pin_21), J_ATX24.22 (Pin_22), J_ATX24.23 (Pin_23), J_ATX24.4 (Pin_4), J_ATX24.6 (Pin_6)
- net GND: now also J_ATX24.15 (Pin_15), J_ATX24.17 (Pin_17), J_ATX24.18 (Pin_18), J_ATX24.19 (Pin_19), J_ATX24.24 (Pin_24), J_ATX24.3 (Pin_3), J_ATX24.5 (Pin_5), J_ATX24.7 (Pin_7), J_EPS8.1 (Pin_1), J_EPS8.2 (Pin_2), J_EPS8.3 (Pin_3), J_EPS8.4 (Pin_4), J_PCIE1.2 (Pin_2), J_PCIE1.4 (Pin_4), J_PCIE1.6 (Pin_6), J_PCIE1.8 (Pin_8), J_PCIE2.2 (Pin_2), J_PCIE2.4 (Pin_4), J_PCIE2.6 (Pin_6), J_PCIE2.8 (Pin_8), J_PWRBTN.2 (Pin_2), J_PWRLED.2 (Pin_2), J_PWROK.2 (Pin_2)
- new net +12V: J_ATX24.10 (Pin_10), J_ATX24.12 (Pin_12), J_EPS8.5 (Pin_5), J_EPS8.6 (Pin_6), J_EPS8.7 (Pin_7), J_EPS8.8 (Pin_8), J_PCIE1.1 (Pin_1), J_PCIE1.3 (Pin_3), J_PCIE1.5 (Pin_5), J_PCIE1.7 (Pin_7), J_PCIE2.1 (Pin_1), J_PCIE2.3 (Pin_3), J_PCIE2.5 (Pin_5), J_PCIE2.7 (Pin_7)
- new net +5VSB: J_ATX24.9 (Pin_9), R8.1
- new net PS_ON: J_ATX24.16 (Pin_16), J_PWRBTN.1 (Pin_1)
- new net PWR_LED_A: J_PWRLED.1 (Pin_1), R8.2
- new net PWR_OK: J_ATX24.8 (Pin_8), J_PWROK.1 (Pin_1)
- no-connect marks 26 -> 29

Commit message: Some updates1
Parts:
- added C10, C13, C16, C8: 100nF, symbol Device:C
- added C11, C14, C17, C7: 560uF, symbol Device:C
- added C12, C15, C6, C9: 10nF, symbol Device:C
- added L1, L2, L3, L4: 220nH, symbol Device:L
- added Q1, Q2, Q3, Q4, Q5, Q6, Q7, Q8: BSC010NE2LS, symbol Device:Q_NMOS
- added R10, R13, R16, R19: 10k, symbol Device:R
- added R11, R14, R17, R20: 4.7k, symbol Device:R
- added R12, R15, R18, R9: 100k, symbol Device:R
- added U3, U4, U5, U6: ISL8117FRZ, symbol Regulator_Switching:ISL8117FRZ
Connections:
- net +12V: now also Q1.D, Q3.D, U3.14 (VIN), U4.14 (VIN), U5.14 (VIN)
- net +5V: now also U3.15 (EXTBIAS), U3.16 (EN), U3.9 (VCC5V), U4.15 (EXTBIAS), U4.16 (EN), U4.9 (VCC5V), U5.15 (EXTBIAS), U5.16 (EN), U5.9 (VCC5V), U6.16 (EN)
- net GND: now also C11.2, C12.2, C14.2, C15.2, C17.2, C6.2, C7.2, C9.2, Q2.S, Q4.S, R11.2, R12.2, R14.2, R15.2, R17.2, R18.2, R20.2, R9.2, U3.17 (SGND), U3.7 (PGND), U4.17 (SGND), U4.7 (PGND), U5.17 (SGND), U5.7 (PGND)
- new net VCORE: C11.1, C14.1, C17.1, C7.1, L1.2, L2.2, L3.2, L4.2, R10.1, R13.1, R16.1, R19.1
- new net VRM_BOOT: C8.1, U3.6 (FB)
- new net VRM_BOOT2: C10.1, U4.6 (FB)
- new net VRM_BOOT3: C13.1, U5.6 (FB)
- new net VRM_BOOT4: C16.1
- new net VRM_CLKOUT: U3.1 (CLKOUT)
- new net VRM_CLKOUT2: U4.1 (CLKOUT)
- new net VRM_CLKOUT3: U5.1 (CLKOUT)
- new net VRM_CLKOUT4: U6.1 (CLKOUT)
- new net VRM_FB: R10.2, R11.1, U3.13 (BOOT)
- new net VRM_FB2: R13.2, R14.1, U4.13 (BOOT)
- new net VRM_FB3: R16.2, R17.1, U5.13 (BOOT)
- new net VRM_FB4: R19.2, R20.1
- new net VRM_ISEN: U3.10 (ISEN)
- new net VRM_ISEN2: U4.10 (ISEN)
- new net VRM_ISEN3: U5.10 (ISEN)
- new net VRM_ISEN4: U6.10 (ISEN)
- new net VRM_LGATE: Q2.G, U3.11 (PHASE)
- new net VRM_LGATE2: Q4.G, U4.11 (PHASE)
- new net VRM_LGATE3: U5.11 (PHASE)
- new net VRM_LGATE4: U6.8 (LGATE/OCS)
- new net VRM_PGOOD: U3.5 (SS/TRK), U4.5 (SS/TRK), U5.5 (SS/TRK)
- new net VRM_PHASE: C8.2, L1.1, Q1.S, Q2.D, U3.8 (LGATE/OCS)
- new net VRM_PHASE2: C10.2, L2.1, Q3.S, Q4.D, U4.8 (LGATE/OCS)
- new net VRM_PHASE3: C13.2, L3.1, U5.8 (LGATE/OCS)
- new net VRM_PHASE4: C16.2, L4.1
- new net VRM_RT: R9.1, U3.2 (MOD/SYNC)
- new net VRM_RT2: R12.1, U4.2 (MOD/SYNC)
- new net VRM_RT3: R15.1, U5.2 (MOD/SYNC)
- new net VRM_RT4: R18.1
- new net VRM_SSTRK: C6.1, U3.3 (PGOOD)
- new net VRM_SSTRK2: C9.1, U4.3 (PGOOD)
- new net VRM_SSTRK3: C12.1, U5.3 (PGOOD)
- new net VRM_SSTRK4: C15.1
- new net VRM_SYNC: U3.4 (RT), U4.4 (RT), U5.4 (RT)
- new net VRM_UGATE: Q1.G, U3.12 (UGATE)
- new net VRM_UGATE2: Q3.G
- new net VRM_UGATE3: U5.12 (UGATE)
- new net VRM_UGATE4: U6.12 (UGATE)
- no-connect marks 29 -> 28

Commit message: Some updates1
Connections:
- net VRM_BOOT4: now also U6.6 (FB)
- net VRM_LGATE3: now also Q6.G
- net VRM_LGATE4: now also Q8.G, U6.11 (PHASE)
- net VRM_PHASE3: now also Q5.S, Q6.D
- net VRM_PHASE4: now also Q7.S, Q8.D
- net VRM_RT4: now also U6.2 (MOD/SYNC)
- net VRM_SSTRK4: now also U6.3 (PGOOD)
- net VRM_UGATE3: now also Q5.G
- net VRM_UGATE4: now also Q7.G
Changed lines of the file:
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@@
 		)
+	)
+	(label "VRM_RT4"
+		(at 274.32 424.18 0)
+		(effects (font (size 1.524 1.524)))
+	)
+	(label "VRM_SSTRK4"
+		(at 274.32 426.72 0)
+		(effects (font (size 1.524 1.524)))
+	)
+	(label "VRM_CLKOUT4"
+		(at 274.32 429.26 0)
+		(effects (font (size 1.524 1.524)))
+	)
+	(label "VRM_UGATE4"
+		(at 304.8 434.34 0)
+		(effects (font (size 1.524 1.524)))
+	)
+	(label "VRM_LGATE4"
+		(at 304.8 426.72 0)
+		(effects (font (size 1.524 1.524)))
+	)
+	(label "VRM_BOOT4"
+		(at 304.8 436.88 0)
+		(effects (font (size 1.524 1.524)))
+	)
+	(label "VRM_UGATE2"
+		(at 325.12 279.4 0)
+		(effects (font (size 1.524 1.524)))
+	)
+	(label "VRM_LGATE2"
+		(at 325.12 299.72 0)
+		(effects (font (size 1.524 1.524)))
+	)
+	(label "VRM_UGATE3"
+		(at 325.12 349.25 0)
+		(effects (font (size 1.524 1.524)))
+	)
+	(label "VRM_LGATE3"
+		(at 325.12 369.57 0)
+		(effects (font (size 1.524 1.524)))
+	)
+	(label "VRM_UGATE4"
+		(at 325.12 419.1 0)
+		(effects (font (size 1.524 1.524)))
+	)
+	(label "VRM_LGATE4"
+		(at 325.12 439.42 0)
+		(effects (font (size 1.524 1.524)))
+	)
+	(label "VRM_PHASE3"
+		(at 332.74 354.33 0)
+		(effects (font (size 1.524 1.524)))
+	)
+	(label "VRM_PHASE3"
+		(at 332.74 364.49 0)
+		(effects (font (size 1.524 1.524)))
+	)
+	(label "VRM_PHASE3"
+		(at 320.04 349.25 0)
+		(effects (font (size 1.524 1.524)))
+	)
+	(label "VRM_PHASE3"
+		(at 355.6 354.33 0)
+		(effects (font (size 1.524 1.524)))
+	)
+	(label "VRM_PHASE4"
+		(at 332.74 424.18 0)
+		(effects (font (size 1.524 1.524)))
+	)
+	(label "VRM_PHASE4"
+		(at 332.74 434.34 0)
+		(effects (font (size 1.524 1.524)))
+	)
+	(label "VRM_PHASE4"
+		(at 320.04 419.1 0)
+		(effects (font (size 1.524 1.524)))
+	)
+	(label "VRM_PHASE4"
+		(at 355.6 424.18 0)
+		(effects (font (size 1.524 1.524)))
+	)
+	(label "VRM_FB4"
+		(at 259.08 450.85 0)
+		(effects (font (size 1.524 1.524)))
+	)
+	(label "VRM_FB4"
+		(at 259.08 453.39 0)
+		(effects (font (size 1.524 1.524)))
 	)
 	(sheet_instances

Commit message: Some updates1
Parts:
- added J_DIMM1, J_DIMM2: DDR4_SO-DIMM_260, symbol dfdtc_Connector:DDR4_SODIMM_CONN260
Connections:
- net +12V: now also Q5.D, Q7.D, U6.14 (VIN)
- net +5V: now also U6.15 (EXTBIAS), U6.9 (VCC5V)
- net GND: now also Q6.S, Q8.S, U6.17 (SGND), U6.7 (PGND)
- net VRM_BOOT4: now also U6.13 (BOOT); no longer U6.6 (FB)
- net VRM_FB4: now also U6.6 (FB)
- net VRM_LGATE4: no longer U6.11 (PHASE)
- net VRM_PGOOD: now also U6.3 (PGOOD)
- net VRM_PHASE4: now also U6.11 (PHASE)
- net VRM_RT4: now also U6.4 (RT); no longer U6.2 (MOD/SYNC)
- net VRM_SSTRK4: now also U6.5 (SS/TRK); no longer U6.3 (PGOOD)
- net VRM_SYNC: now also U6.2 (MOD/SYNC)
- net VRM_UGATE2: now also U4.12 (UGATE)
